Commit message: update the code base

File: surrol/assets/block/block.urdf (robot description, URDF)
Before this commit: robot block, 4 links, 3 joints
Links:
- link baseLink: mass 0.01 -> 1

File: surrol/assets/needle/needle_40mm.urdf (robot description, URDF)
Before this commit: robot needle, 7 links, 6 joints
Links:
- link baseLink: mass 0.01 -> 0.51

File: surrol/assets/peg_board/peg_board.urdf (robot description, URDF)
Before this commit: robot peg_board, 13 links, 12 joints
Links:
- link baseLink: mass .0 -> 100.0
- link peg_1: mass .0 -> 100.0; geometry collision cylinder length=0.0168 radius=0.001; visual mesh filename=meshes/peg.obj scale=1 1 0.6
- link peg_10: mass .0 -> 100.0; geometry collision cylinder length=0.0168 radius=0.001; visual mesh filename=meshes/peg.obj scale=1 1 0.6
- link peg_11: mass .0 -> 100.0; geometry collision cylinder length=0.0168 radius=0.001; visual mesh filename=meshes/peg.obj scale=1 1 0.6
- link peg_12: mass .0 -> 100.0; geometry collision cylinder length=0.0168 radius=0.001; visual mesh filename=meshes/peg.obj scale=1 1 0.6
- link peg_2: mass .0 -> 100.0; geometry collision cylinder length=0.0168 radius=0.001; visual mesh filename=meshes/peg.obj scale=1 1 0.6
- link peg_3: mass .0 -> 100.0; geometry collision cylinder length=0.0168 radius=0.001; visual mesh filename=meshes/peg.obj scale=1 1 0.6
- link peg_4: mass .0 -> 100.0; geometry collision cylinder length=0.0168 radius=0.001; visual mesh filename=meshes/peg.obj scale=1 1 0.6
- link peg_5: mass .0 -> 100.0; geometry collision cylinder length=0.0168 radius=0.001; visual mesh filename=meshes/peg.obj scale=1 1 0.6
- link peg_6: mass .0 -> 100.0; geometry collision cylinder length=0.0168 radius=0.001; visual mesh filename=meshes/peg.obj scale=1 1 0.6
- link peg_7: mass .0 -> 100.0; geometry collision cylinder length=0.0168 radius=0.001; visual mesh filename=meshes/peg.obj scale=1 1 0.6
- link peg_8: mass .0 -> 100.0; geometry collision cylinder length=0.0168 radius=0.001; visual mesh filename=meshes/peg.obj scale=1 1 0.6
- link peg_9: mass .0 -> 100.0; geometry collision cylinder length=0.0168 radius=0.001; visual mesh filename=meshes/peg.obj scale=1 1 0.6

File: surrol/assets/psm/psm.urdf (robot description, URDF)
Before this commit: robot psm, 17 links, 16 joints
Links:
- link psm_main_insertion_link_3: geometry visual mesh filename=meshes/visual/CDF_base.obj scale=0.001 0.001 0.001
- link psm_tool_gripper1_link: mass 0.02 -> 2.02
- link psm_tool_gripper2_link: mass 0.02 -> 2.02
- link psm_tool_pitch_link: geometry collision mesh filename=meshes/collision/wrist.obj scale=0.001 0.001 0.001; visual mesh filename=meshes/visual/wrist.obj scale=0.001 0.001 0.001
- link psm_tool_roll_link: geometry collision mesh filename=meshes/collision/CDF_base_no_shaft.obj scale=0.001 0.001 0.001; visual mesh filename=meshes/visual/CDF_base_no_shaft.obj scale=0.001 0.001 0.001
- link psm_tool_yaw_link: geometry 
Joints:
- joint psm_main_insertion_joint: limit lower=0 upper=0.24 effort=100 velocity=1 -> lower=0 upper=0.24 effort=200 velocity=1
- joint psm_pitch_back_joint: limit lower=-0.93556 upper=0.94249 effort=100 velocity=10 -> lower=-0.93556 upper=0.94249 effort=200 velocity=10
- joint psm_pitch_bottom_joint: limit lower=-0.94249 upper=0.93556 effort=100 velocity=10 -> lower=-0.94249 upper=0.93556 effort=200 velocity=10
- joint psm_pitch_end_joint: limit lower=-0.9251 upper=0.9251 effort=100 velocity=2.1 -> lower=-0.9251 upper=0.9251 effort=200 velocity=2.1
- joint psm_pitch_front_joint: limit lower=-0.93556 upper=0.94249 effort=100 velocity=10 -> lower=-0.93556 upper=0.94249 effort=200 velocity=10
- joint psm_pitch_top_joint: limit lower=-0.94249 upper=0.93556 effort=100 velocity=10 -> lower=-0.94249 upper=0.93556 effort=200 velocity=10
- joint psm_tool_gripper1_joint: limit lower=-1 upper=1 effort=20 velocity=2.1 -> lower=-1 upper=1 effort=200 velocity=2.1
- joint psm_tool_gripper2_joint: limit lower=-1 upper=1 effort=20 velocity=2.1 -> lower=-1 upper=1 effort=200 velocity=2.1
- joint psm_tool_pitch_joint: limit lower=-1.3963 upper=1.3963 effort=100 velocity=2.1 -> lower=-1.3963 upper=1.3963 effort=200 velocity=2.1
- joint psm_tool_roll_joint: limit lower=-4.5379 upper=4.5379 effort=100 velocity=2.1 -> lower=-4.5379 upper=4.5379 effort=200 velocity=2.1
- joint psm_tool_yaw_joint: limit lower=-1.3963 upper=1.3963 effort=100 velocity=2.1 -> lower=-1.3963 upper=1.3963 effort=200 velocity=21
- joint psm_yaw_joint: limit lower=-1.5883 upper=1.5883 effort=100 velocity=2.1 -> lower=-1.5883 upper=1.5883 effort=200 velocity=2.1

File: surrol/assets/tray/pad.urdf (robot description, URDF)
Before this commit: robot pad, 1 links, 0 joints
Links:
- link baseLink: mass .0 -> 100.0

File: surrol/assets/tray/tray.urdf (robot description, URDF)
Before this commit: robot tray, 5 links, 4 joints
Links:
- link baseLink: mass .0 -> 100.0
- link border_1: mass .0 -> 10.0
- link border_2: mass .0 -> 10.0
- link border_3: mass .0 -> 10.0
- link border_4: mass .0 -> 10.0

File: surrol/assets/tray/tray_pad.urdf (robot description, URDF)
Before this commit: robot tray, 6 links, 5 joints
Links:
- link baseLink: mass .0 -> 0.01
- link border_1: mass .0 -> 100.0; geometry collision box size=0.120 0.003 0.025; visual box size=0 0 0
- link border_2: mass .0 -> 100.0; geometry collision box size=0.120 0.003 0.025; visual box size=0 0 0
- link border_3: mass .0 -> 100.0; geometry collision box size=0.003 0.196 0.025; visual box size=0 0 0
- link border_4: mass .0 -> 100.0; geometry collision box size=0.003 0.196 0.025; visual box size=0 0 0
- link pad: mass .0 -> 0.01
